File: KRONE_Controller/Hardware/Fallblatt-Controller.kicad_pcb (KiCad board)
At the start: 2 copper layers, 100 x 62 mm, 39 parts, among them P1 ISP, P2 Motor, P3 Interface, P4 42V AC, Q1 MOC3081M, Q2 BC817-40, Q3 BC817-40, SW1 DM-08-V, U1 ATMEGA328PB-AN, U2 MAX485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

Commit message: Some old hardware changes for v1.1
Parts:
- U1: value ATMEGA328PB-AN -> ATMEGA328P-AU
Connections:
- P3 pad 5: /AUX2 -> GND
- P3 pad 6: /AUX1 -> +5V
- U1 pad 3: /AUX1 -> GND
- U1 pad 6: /AUX2 -> +5V
Routing:
- net /AUX2: track 49.8 -> 0.00 mm, vias 2 -> 0
- net /AUX1: track 44.7 -> 0.00 mm, vias 1 -> 0
- net +5V: track 196.8 -> 203.2 mm
- net GND: track 26.0 -> 28.3 mm
