File: KRONE_Controller/Hardware/Fallblatt-Controller.sch (KiCad schematic (older format))
At the start: 25 parts, among them P1 ISP, P2 Motor, P3 Interface, P4 42V AC, Q1 MOC3081M, Q2 BC817-40, Q3 BC817-40, SW1 DM-08-V, U1 ATMEGA328P-AU, U2 MAX485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

Commit message: Some old hardware changes for v1.1
Connections:
- net +5V: now also P3.6 (P6), U1.6 (PE1(PTCXY/SCL1/T4))
- net GND: now also P3.5 (P5), U1.3 (PE0(PTCXY/SDA1/ICP4/ACO))
- removed net AUX1: P3.6 (P6), U1.3 (PE0(PTCXY/SDA1/ICP4/ACO))
- removed net AUX2: P3.5 (P5), U1.6 (PE1(PTCXY/SCL1/T4))
Other:
- note added: "Diese beiden Pins sind KEINE IO-Pins!"
Changed lines of the file:
@@
 Sheet 1 1
 Title "Fallblatt-Controller"
-Date "2017-09-25"
-Rev "v1.0"
+Date "2017-10-14"
+Rev "v1.1"
 Comp "xatLabs"
 Comment1 "Julian Metzler"
@@
 	1    0    0    -1
 $EndComp
-Text Notes 10950 6850 2    60   ~ 0
+Text Notes 11150 7250 2    60   ~ 0
 Nur beim letzten Modul
 $Comp
@@
 NoConn ~ 5900 6050
 NoConn ~ 5900 6150
-NoConn ~ 8500 6350
-NoConn ~ 8500 6450
 $Comp
 L C C2
@@
 	12150 7100 12150 6950
 Connection ~ 11450 7100
-Text Label 11700 6400 0    60   ~ 0
-AUX1
-Wire Wire Line
-	11700 6400 11550 6400
-Wire Wire Line
-	11550 6400 11550 6550
-Text Label 11700 7200 0    60   ~ 0
-AUX2
-Wire Wire Line
-	11700 7200 11550 7200
-Wire Wire Line
-	11550 7200 11550 7050
 $Comp
 L R R4
@@
 $EndComp
 Connection ~ 6900 3500
-Text Label 5900 5850 2    60   ~ 0
-AUX1
-Text Label 5900 5950 2    60   ~ 0
-AUX2
 $Comp
 L +5V #PWR018
@@
 Wire Wire Line
 	8650 6250 8500 6250
+$Comp
+L +5V #PWR?
+U 1 1 59E1DB0F
+P 5750 5800
+F 0 "#PWR?" H 5750 5650 50  0001 C CNN
+F 1 "+5V" H 5765 5973 50  0000 C CNN
+F 2 "" H 5750 5800 50  0000 C CNN
+F 3 "" H 5750 5800 50  0000 C CNN
+	1    5750 5800
+	1    0    0    -1
+$EndComp
+$Comp
+L GND #PWR?
+U 1 1 59E1DB55
+P 5800 6200
+F 0 "#PWR?" H 5800 5950 50  0001 C CNN
+F 1 "GND" H 5805 6027 50  0000 C CNN
+F 2 "" H 5800 6200 50  0000 C CNN
+F 3 "" H 5800 6200 50  0000 C CNN
+	1    5800 6200
+	1    0    0    -1
+$EndComp
+Wire Wire Line
+	5800 6200 5800 5850
+Wire Wire Line
+	5800 5850 5900 5850
+Wire Wire Line
+	5750 5800 5750 5950
+Wire Wire Line
+	5750 5950 5900 5950
+Text Notes 6100 5700 0    60   ~ 0
+Diese beiden Pins sind KEINE IO-Pins!
+Wire Notes Line
+	6150 5700 6150 5800
+Wire Notes Line
+	10850 7150 10850 6800
+Wire Notes Line
+	10850 6800 10950 6800
+NoConn ~ 8500 6350
+NoConn ~ 8500 6450
+Wire Wire Line
+	11550 6550 11550 6500
+Connection ~ 11550 6500
+Wire Wire Line
+	11550 7050 11550 7100
+Connection ~ 11550 7100
 $EndSCHEMATC

Commit message: Updated splitflap controller schematic to new kicad version
Parts:
- C1, C2: symbol C -> Fallblatt-Controller-rescue:C
- C3: symbol CP -> Fallblatt-Controller-rescue:CP
- D1: symbol Q_TRIAC_AAG_Alternate -> Fallblatt-Controller-rescue:Q_TRIAC_AAG_Alternate
- D2, D3: symbol Photointerrupter -> Fallblatt-Controller-rescue:Photointerrupter
- P1, P3: symbol CONN_02X03 -> Fallblatt-Controller-rescue:CONN_02X03
- P2, P4: symbol CONN_01X02 -> Fallblatt-Controller-rescue:CONN_01X02
- Q1: symbol MOC3081M -> Fallblatt-Controller-rescue:MOC3081M
- Q2, Q3: symbol BC817-40 -> Fallblatt-Controller-rescue:BC817-40
- R1, R2, R3, R4, R5, R6, R7, R8: symbol R -> Fallblatt-Controller-rescue:R
- SW1: symbol SW_DIP_x08 -> Fallblatt-Controller-rescue:SW_DIP_x08
- U1: symbol ATMEGA328PB-AU -> Fallblatt-Controller-rescue:ATMEGA328PB-AU
- U2: symbol SP3481EN -> Fallblatt-Controller-rescue:SP3481EN
- Y1: symbol Resonator -> Fallblatt-Controller-rescue:Resonator
